File: AmpSwitchAutomatic_control.brd (EAGLE design)
At the start: 127 x 61 mm, 57 parts, among them IC1 LM339N, IC2 4051N, IC3 NE555, IC4 7493N-MM74C, IC5 4035N, IC6 4035N, IC7 4585N, IC8 74132N, Q1 BS170DGS

Commit message: Finalized
Parts:
- added C8: 100nF, rcl:C050-025X075
- added J1: POWER_JACKPTH_BREAD, SparkFun-Connectors:POWER_JACK_PTH_BREAD
- added JP1, JP2: (no value), pinhead:1X01
- moved LED1 16.3 mm to (104.1, 67.3)
- moved PAD14 14.8 mm to (50.8, 63.5)
- moved R14 13.7 mm to (63.5, 49.5)
- moved D1 13.0 mm to (58.4, 58.4)
- moved Q1 13.0 mm to (111.8, 58.4)
- moved D2 12.7 mm to (33.0, 54.6)
- moved IC8 12.7 mm to (44.5, 58.4)
- moved PAD12 12.7 mm to (25.4, 55.9)
- moved PAD15 12.7 mm to (25.4, 53.3)
- moved PAD16 12.7 mm to (10.2, 71.1)
- moved PAD17 12.7 mm to (10.2, 66.0)
- moved PAD7 12.7 mm to (119.4, 33.0)
- moved R12 12.7 mm to (101.6, 49.5)
- moved R13 12.7 mm to (73.7, 54.6)
- moved R15 12.7 mm to (35.6, 47.0)
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Connections:
- net GND: now also C8.2, J1.GND
- net N$20: now also C8.1
- net VCC: now also J1.PWR
Routing:
- net CNT_0: track 183.5 -> 129.5 mm
- net CNT_1: track 191.9 -> 139.7 mm
- net CNT_2: track 159.6 -> 111.8 mm
- net VCC: track 430.7 -> 438.3 mm
- net N$17: track 40.6 -> 48.3 mm
- net AUDIO6: track 40.6 -> 35.0 mm
- net CLK: track 175.3 -> 172.7 mm
- net SIGNAL_L: track 25.4 -> 22.9 mm
- net RESET_LATCH: track 7.62 -> 5.08 mm
- net N$5: track 7.62 -> 5.08 mm
- net PRESENT_ST_2: track 55.9 -> 54.4 mm
