File: AmpSwitchAutomatic_control.sch (EAGLE design)
At the start: 57 parts, among them IC1 LM339N, IC2 4051N, IC3 NE555, IC4 7493N-MM74C, IC5 4035N, IC6 4035N, IC7 4585N, IC8 74132N, Q1 BS170DGS

Commit message: Finalized
Parts:
- added C8: 100nF, rcl:C-EU050-025X075
- added J1: POWER_JACKPTH_BREAD, SparkFun-Connectors:POWER_JACKPTH_BREAD
- added JP1, JP2: (no value), pinhead:PINHD-1X1
Connections:
- net GND: now also C8.2, J1.GND
- net N$20: now also C8.1
- net VCC: now also J1.PWR
