File: AmpSwitchAutomatic_main.brd (EAGLE design)
At the start: 149.9 x 81.3 mm, 81 parts, among them IC1 4051N, K1L DS2Y-S-DC9V, K1R DS2Y-S-DC9V, K2L DS2Y-S-DC9V, K2R DS2Y-S-DC9V, K3L DS2Y-S-DC9V, K3R DS2Y-S-DC9V, K4L DS2Y-S-DC9V, K4R DS2Y-S-DC9V, K5L DS2Y-S-DC9V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

Commit message: Finalized
Parts:
- added D10, D11, D12, D13, D14, D15, D16, D17, D18, D7, D8, D9: (no value), diode:ZDIO-7.5
- added JP1, JP2: (no value), pinhead:1X01
Connections:
- net AUDIO1: now also D7.C, D8.A
- net AUDIO2: now also D10.A, D9.C
- net AUDIO3: now also D11.C, D12.A
- net AUDIO4: now also D13.C, D14.A
- net AUDIO5: now also D15.C, D16.A
- net AUDIO6: now also D17.C, D18.A
- net GND: now also D10.C, D11.A, D12.C, D13.A, D14.C, D15.A, D16.C, D17.A, D18.C, D7.A, D8.C, D9.A
Changed lines of the file:
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@@
 <element name="PAD34" library="wirepad" package="2,15/1,0" value="" x="116.84" y="43.18"/>
 <element name="PAD35" library="wirepad" package="2,15/1,0" value="" x="116.84" y="55.88"/>
+<element name="JP1" library="pinhead" package="1X01" value="" x="0" y="66.04"/>
+<element name="JP2" library="pinhead" package="1X01" value="" x="2.54" y="30.48"/>
+<element name="D7" library="diode" package="ZDIO-7.5" value="" x="5.08" y="-5.08"/>
+<element name="D8" library="diode" package="ZDIO-7.5" value="" x="5.08" y="-10.16" rot="R180"/>
+<element name="D9" library="diode" package="ZDIO-7.5" value="" x="17.78" y="-5.08"/>
+<element name="D10" library="diode" package="ZDIO-7.5" value="" x="17.78" y="-10.16" rot="R180"/>
+<element name="D11" library="diode" package="ZDIO-7.5" value="" x="30.48" y="-5.08"/>
+<element name="D12" library="diode" package="ZDIO-7.5" value="" x="30.48" y="-10.16" rot="R180"/>
+<element name="D13" library="diode" package="ZDIO-7.5" value="" x="43.18" y="-5.08"/>
+<element name="D14" library="diode" package="ZDIO-7.5" value="" x="43.18" y="-10.16" rot="R180"/>
+<element name="D15" library="diode" package="ZDIO-7.5" value="" x="55.88" y="-5.08"/>
+<element name="D16" library="diode" package="ZDIO-7.5" value="" x="55.88" y="-10.16" rot="R180"/>
+<element name="D17" library="diode" package="ZDIO-7.5" value="" x="68.58" y="-5.08"/>
+<element name="D18" library="diode" package="ZDIO-7.5" value="" x="68.58" y="-10.16" rot="R180"/>
 </elements>
 <signals>
@@
 <wire x1="137.16" y1="30.48" x2="138.43" y2="29.21" width="0.4064" layer="1"/>
 <wire x1="138.43" y1="29.21" x2="137.16" y2="27.94" width="0.4064" layer="1"/>
+<contactref element="D7" pad="A"/>
+<contactref element="D8" pad="C"/>
+<contactref element="D17" pad="A"/>
+<contactref element="D18" pad="C"/>
+<contactref element="D15" pad="A"/>
+<contactref element="D16" pad="C"/>
+<contactref element="D13" pad="A"/>
+<contactref element="D14" pad="C"/>
+<contactref element="D11" pad="A"/>
+<contactref element="D12" pad="C"/>
+<contactref element="D9" pad="A"/>
+<contactref element="D10" pad="C"/>
+<wire x1="72.39" y1="-5.08" x2="72.39" y2="-10.16" width="0" layer="19" extent="1-1"/>
+<wire x1="59.69" y1="-10.16" x2="72.39" y2="-5.08" width="0" layer="19" extent="1-1"/>
+<wire x1="59.69" y1="-5.08" x2="59.69" y2="-10.16" width="0" layer="19" extent="1-1"/>
+<wire x1="46.99" y1="-10.16" x2="59.69" y2="-5.08" width="0" layer="19" extent="1-1"/>
+<wire x1="46.99" y1="-5.08" x2="46.99" y2="-10.16" width="0" layer="19" extent="1-1"/>
+<wire x1="34.29" y1="-10.16" x2="46.99" y2="-5.08" width="0" layer="19" extent="1-1"/>
+<wire x1="34.29" y1="-5.08" x2="34.29" y2="-10.16" width="0" layer="19" extent="1-1"/>
+<wire x1="21.59" y1="-10.16" x2="34.29" y2="-5.08" width="0" layer="19" extent="1-1"/>
+<wire x1="21.59" y1="-5.08" x2="21.59" y2="-10.16" width="0" layer="19" extent="1-1"/>
+<wire x1="8.89" y1="-10.16" x2="21.59" y2="-5.08" width="0" layer="19" extent="1-1"/>
+<wire x1="8.89" y1="-5.08" x2="8.89" y2="-10.16" width="0" layer="19" extent="1-1"/>
+<wire x1="10.16" y1="10.16" x2="8.89" y2="-5.08" width="0" layer="19" extent="1-1"/>
 </signal>
 <signal name="AUDIO1">
@@
 <contactref element="SV2" pad="7"/>
 <wire x1="121.92" y1="25.4" x2="24.13" y2="25.4" width="1.27" layer="16"/>
+<contactref element="D7" pad="C"/>
+<contactref element="D8" pad="A"/>
+<wire x1="1.27" y1="-5.08" x2="24.13" y2="25.4" width="0" layer="19" extent="1-1"/>
+<wire x1="1.27" y1="-10.16" x2="1.27" y2="-5.08" width="0" layer="19" extent="1-1"/>
 </signal>
 <signal name="AUDIO2">
@@
 <contactref element="SV2" pad="8"/>
 <wire x1="121.92" y1="22.86" x2="41.91" y2="22.86" width="1.27" layer="16"/>
+<contactref element="D10" pad="A"/>
+<contactref element="D9" pad="C"/>
+<wire x1="13.97" y1="-10.16" x2="41.91" y2="22.86" width="0" layer="19" extent="1-1"/>
+<wire x1="13.97" y1="-5.08" x2="13.97" y2="-10.16" width="0" layer="19" extent="1-1"/>
 </signal>
 <signal name="AUDIO3">
@@
 <contactref element="SV2" pad="9"/>
 <wire x1="121.92" y1="20.32" x2="59.69" y2="20.32" width="1.27" layer="16"/>
+<contactref element="D12" pad="A"/>
+<contactref element="D11" pad="C"/>
+<wire x1="26.67" y1="-10.16" x2="59.69" y2="20.32" width="0" layer="19" extent="1-1"/>
+<wire x1="26.67" y1="-5.08" x2="26.67" y2="-10.16" width="0" layer="19" extent="1-1"/>
 </signal>
 <signal name="AUDIO4">
@@
 <contactref element="SV2" pad="10"/>
 <wire x1="121.92" y1="17.78" x2="76.2" y2="17.78" width="1.27" layer="16"/>
+<contactref element="D14" pad="A"/>
+<contactref element="D13" pad="C"/>
+<wire x1="39.37" y1="-10.16" x2="76.2" y2="17.78" width="0" layer="19" extent="1-1"/>
+<wire x1="39.37" y1="-5.08" x2="39.37" y2="-10.16" width="0" layer="19" extent="1-1"/>
 </signal>
 <signal name="AUDIO5">
@@
 <contactref element="SV2" pad="11"/>
 <wire x1="121.92" y1="15.24" x2="111.76" y2="15.24" width="1.27" layer="16"/>
+<contactref element="D16" pad="A"/>
+<contactref element="D15" pad="C"/>
+<wire x1="52.07" y1="-10.16" x2="93.98" y2="15.24" width="0" layer="19" extent="1-1"/>
+<wire x1="52.07" y1="-5.08" x2="52.07" y2="-10.16" width="0" layer="19" extent="1-1"/>
 </signal>
 <signal name="AUDIO6">
@@
 <wire x1="121.92" y1="12.7" x2="116.84" y2="12.7" width="1.27" layer="16"/>
 <wire x1="147.32" y1="12.7" x2="121.92" y2="12.7" width="1.27" layer="16"/>
+<contactref element="D17" pad="C"/>
+<contactref element="D18" pad="A"/>
+<wire x1="64.77" y1="-10.16" x2="116.84" y2="12.7" width="0" layer="19" extent="1-1"/>
+<wire x1="64.77" y1="-5.08" x2="64.77" y2="-10.16" width="0" layer="19" extent="1-1"/>
 </signal>
 <signal name="N$23">
