File: AmpSwitchAutomatic_main.sch (EAGLE design)
At the start: 81 parts, among them IC1 4051N, K1L DS2Y-S-DC9V, K1R DS2Y-S-DC9V, K2L DS2Y-S-DC9V, K2R DS2Y-S-DC9V, K3L DS2Y-S-DC9V, K3R DS2Y-S-DC9V, K4L DS2Y-S-DC9V, K4R DS2Y-S-DC9V, K5L DS2Y-S-DC9V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

Commit message: Finalized
Parts:
- added D10, D11, D12, D13, D14, D15, D16, D17, D18, D7, D8, D9: (no value), diode:ZENER-DIODEZD-7.5
- added JP1, JP2: (no value), pinhead:PINHD-1X1
Connections:
- net AUDIO1: now also D7.C, D8.A
- net AUDIO2: now also D10.A, D9.C
- net AUDIO3: now also D11.C, D12.A
- net AUDIO4: now also D13.C, D14.A
- net AUDIO5: now also D15.C, D16.A
- net AUDIO6: now also D17.C, D18.A
- net GND: now also D10.C, D11.A, D12.C, D13.A, D14.C, D15.A, D16.C, D17.A, D18.C, D7.A, D8.C, D9.A
